Commit message: add laser scan matcher

File: chusa_bringup/robot_base/urdf/chusa_bot.urdf (robot description, URDF)
Before this commit: robot robot, 12 links, 11 joints
Links:
- removed link base_scan
- added link laser, mass 0.213; collision box size=0.1 0.075 0.06; visual box size=0.1 0.075 0.06
Joints:
- joint base_scan_joint: child base_scan -> laser

Commit message: sibal

File: chusa_bringup/robot_base/urdf/chusa_bot.urdf (robot description, URDF)
Before this commit: robot robot, 12 links, 11 joints
Joints:
- joint base_scan_joint: origin xyz=0.05 0 0.0545 -> xyz=0.05 0 0.0545 rpy=0 0 1.57
